File: kicad/attops2adapter.kicad_pcb (KiCad board)
At the start: 2 copper layers, 23.8 x 35 mm, 4 parts, among them J1 Mini-DIN-6

Commit message: Rev 0.1 board
Other:
- board text added: "AT ⇄ PS/2 ADAPTER"
- board text removed: "PS/2 ⇄ AT ADAPTER"
Changed lines of the file:
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@@
 		)
 	)
-	(gr_text "PS/2 ⇄ AT ADAPTER"
+	(gr_text "AT ⇄ PS/2 ADAPTER"
 		(at 32 16.1 0)
 		(layer "B.SilkS")
